Commit message: added imu with ROS 2

File: robot_description/urdf/yuna.urdf (robot description, URDF)
Before this commit: robot m6, 42 links, 41 joints
Links:
- removed link realsense_d435_camera_bottom_screw_frame
- removed link realsense_d435_camera_color_frame
- removed link realsense_d435_camera_color_optical_frame
- removed link realsense_d435_camera_depth_frame
- removed link realsense_d435_camera_depth_optical_frame
- removed link realsense_d435_camera_left_ir_frame
- removed link realsense_d435_camera_left_ir_optical_frame
- removed link realsense_d435_camera_link
- removed link realsense_d435_camera_right_ir_frame
- removed link realsense_d435_camera_right_ir_optical_frame
- link base1__INPUT_INTERFACE: geometry collision box size=0.106400 0.069500 0.031050; visual mesh filename=package://robot_description/meshes/M6_base_motor.STL
- link base2__INPUT_INTERFACE: geometry collision box size=0.106400 0.069500 0.031050; visual mesh filename=package://robot_description/meshes/M6_base_motor.STL
- link base3__INPUT_INTERFACE: geometry collision box size=0.106400 0.069500 0.031050; visual mesh filename=package://robot_description/meshes/M6_base_motor.STL
- link base4__INPUT_INTERFACE: geometry collision box size=0.106400 0.069500 0.031050; visual mesh filename=package://robot_description/meshes/M6_base_motor.STL
- link base5__INPUT_INTERFACE: geometry collision box size=0.106400 0.069500 0.031050; visual mesh filename=package://robot_description/meshes/M6_base_motor.STL
- link base6__INPUT_INTERFACE: geometry collision box size=0.106400 0.069500 0.031050; visual mesh filename=package://robot_description/meshes/M6_base_motor.STL
- link base_link: geometry collision box size=0.073 0.075 0.046; collision box size=0.073 0.075 0.046
- link camera_mount: geometry collision mesh filename=package://robot_description/meshes/camera_mount.STL scale=1 1 1; visual mesh filename=package://robot_description/meshes/camera_mount.STL scale=1 1 1
- link elbow1__INPUT_INTERFACE: geometry collision box size=0.05950 0.04800 0.037500; collision box size=0.06850 0.06500 0.037500
- link elbow2__INPUT_INTERFACE: geometry collision box size=0.05950 0.04800 0.037500; collision box size=0.06850 0.06500 0.037500
- link elbow3__INPUT_INTERFACE: geometry collision box size=0.05950 0.04800 0.037500; collision box size=0.06850 0.06500 0.037500
- link elbow4__INPUT_INTERFACE: geometry collision box size=0.05950 0.04800 0.037500; collision box size=0.06850 0.06500 0.037500
- link elbow5__INPUT_INTERFACE: geometry collision box size=0.05950 0.04800 0.037500; collision box size=0.06850 0.06500 0.037500
- link elbow6__INPUT_INTERFACE: geometry collision box size=0.05950 0.04800 0.037500; collision box size=0.06850 0.06500 0.037500
- link leg1__LAST_LINK: geometry collision box size=0.045000 0.047030 0.047030; collision box size=0.05850 0.04800 0.03650
- link leg2__LAST_LINK: geometry collision box size=0.045000 0.047030 0.047030; collision box size=0.05850 0.04800 0.03650
- link leg3__LAST_LINK: geometry collision box size=0.045000 0.047030 0.047030; collision box size=0.05850 0.04800 0.03650
- link leg4__LAST_LINK: geometry collision box size=0.045000 0.047030 0.047030; collision box size=0.05850 0.04800 0.03650
- link leg5__LAST_LINK: geometry collision box size=0.045000 0.047030 0.047030; collision box size=0.05850 0.04800 0.03650
- link leg6__LAST_LINK: geometry collision box size=0.045000 0.047030 0.047030; collision box size=0.05850 0.04800 0.03650
- link shoulder1__INPUT_INTERFACE: geometry collision box size=0.108140 0.04500 0.104000; visual mesh filename=package://robot_description/meshes/M6_left_link1_red.STL
- link shoulder2__INPUT_INTERFACE: geometry collision box size=0.108140 0.04500 0.104000; visual mesh filename=package://robot_description/meshes/M6_right_link1_red.STL
- link shoulder3__INPUT_INTERFACE: geometry collision box size=0.108140 0.04500 0.104000; visual mesh filename=package://robot_description/meshes/M6_left_link1_red.STL
- link shoulder4__INPUT_INTERFACE: geometry collision box size=0.108140 0.04500 0.104000; visual mesh filename=package://robot_description/meshes/M6_right_link1_red.STL
- link shoulder5__INPUT_INTERFACE: geometry collision box size=0.108140 0.04500 0.104000; visual mesh filename=package://robot_description/meshes/M6_left_link1_red.STL
- link shoulder6__INPUT_INTERFACE: geometry collision box size=0.108140 0.04500 0.104000; visual mesh filename=package://robot_description/meshes/M6_right_link1_red.STL
Joints:
- removed joint realsense_d435_camera_color_joint
- removed joint realsense_d435_camera_color_optical_joint
- removed joint realsense_d435_camera_depth_joint
- removed joint realsense_d435_camera_depth_optical_joint
- removed joint realsense_d435_camera_joint
- removed joint realsense_d435_camera_left_ir_joint
- removed joint realsense_d435_camera_left_ir_optical_joint
- removed joint realsense_d435_camera_link_joint
- removed joint realsense_d435_camera_right_ir_joint
- removed joint realsense_d435_camera_right_ir_optical_joint
